Commit message: update

File: assets/urdf/shadow_hand_description/shadowhand_with_fingertips.urdf (robot description, URDF)
Before this commit: robot shadowhand_motor, 30 links, 29 joints
Links:
- added link base_link
- added link pitch_link
- added link roll_link
- added link translation_x
- added link translation_y
- added link translation_z
- added link yaw_link
Joints:
- added joint pitch_joint: type revolute, parent roll_link, child pitch_link, origin xyz=0 0 0 rpy=0 0 0, axis 0 1 0, limit lower=-3.1415926 upper=3.1415926 effort=5 velocity=1.0
- added joint prismatic_joint_x: type prismatic, parent base_link, child translation_x, origin xyz=0 0 0, axis 1 0 0, limit lower=-2 upper=2 effort=5.0 velocity=0.1
- added joint prismatic_joint_y: type prismatic, parent translation_x, child translation_y, origin xyz=0 0 0, axis 0 1 0, limit lower=-2 upper=2 effort=5.0 velocity=0.1
- added joint prismatic_joint_z: type prismatic, parent translation_y, child translation_z, origin xyz=0 0 0, axis 0 0 1, limit lower=-2 upper=2 effort=5.0 velocity=0.1
- added joint roll_joint: type revolute, parent translation_z, child roll_link, origin xyz=0 0 0 rpy=0 0 0, axis 1 0 0, limit lower=-3.1415926 upper=3.1415926 effort=5 velocity=1.0
- added joint yaw_joint: type revolute, parent pitch_link, child forearm, origin xyz=0 0 0 rpy=0 0 0, axis 0 0 1, limit lower=-3.1415926 upper=3.1415926 effort=5 velocity=1.0
