Commit message: finish left hand visual,

File: assets/urdf/shadow_hand/shadow_hand_left.urdf (robot description, URDF)
Before this commit: robot bimanual_shadowhand_motor, 32 links, 31 joints
Links:
- link lfdistal: geometry collision mesh filename=meshes/visual/f_distal/pst/f_distal_pst.dae scale=0.001 0.001 0.001; visual mesh filename=meshes/visual/f_distal/pst/f_distal_pst.dae scale=0.001 0.001 0.001
- link lfknuckle: geometry collision cylinder length=0.014 radius=0.007; visual mesh filename=meshes/visual/f_knuckle/f_knuckle_E3M5.dae scale=0.001 0.001 0.001
- link lfmetacarpal: geometry collision box size=0.018 0.024 0.040; visual mesh filename=meshes/visual/lf_metacarpal/lf_metacarpal_E3M5_left.dae scale=0.001 0.001 0.001
- link lfmiddle: geometry collision cylinder length=0.025 radius=0.007; collision sphere radius=0.007
- link lfproximal: geometry collision cylinder length=0.040 radius=0.007; visual mesh filename=meshes/visual/f_proximal/f_proximal_E3M5.dae scale=0.001 0.001 0.001
- link thbase: geometry collision sphere radius=0.011; visual box size=0.001 0.001 0.001
- link thdistal: geometry collision mesh filename=meshes/visual/th_distal/pst/th_distal_pst.dae scale=0.001 0.001 0.001; visual mesh filename=meshes/visual/th_distal/pst/th_distal_pst.dae scale=0.001 0.001 0.001
- link thhub: geometry collision sphere radius=0.010; visual box size=0.001 0.001 0.001
- link thmiddle: geometry collision cylinder length=0.014 radius=0.010; collision cylinder length=0.018 radius=0.011
- link thproximal: geometry collision cylinder length=0.018 radius=0.012; visual mesh filename=meshes/visual/th_proximal/th_proximal_E3M5.dae scale=0.001 0.001 0.001
Joints:
- joint LFJ5: axis 1 0 0 -> 0 0 -1
- joint THJ5: origin xyz=0.034 -0.00858 0.029 rpy=-0.785398163397 0 -1.57079632679 -> xyz=-0.034 -0.00858 0.029 rpy=-0.785398163397 0 1.57079632679

File: assets/urdf/shadow_hand/shadow_hand_right.urdf (robot description, URDF)
Before this commit: robot bimanual_shadowhand_motor, 32 links, 31 joints
Joints:
- joint LFJ5: axis 1 0 0 -> 0 1 0

Commit message: left thumb not accurate

File: assets/urdf/shadow_hand/shadow_hand_left.urdf (robot description, URDF)
Before this commit: robot bimanual_shadowhand_motor, 32 links, 31 joints
Joints:
- joint palm_to_imu: origin xyz=0.01785 0.00765 0.049125 rpy=-1.5707963 3.141592 0.0 -> xyz=-0.01785 0.00765 0.049125 rpy=-1.5707963 3.141592 0.0

File: assets/urdf/shadow_hand/shadow_hand_left_collision.urdf (robot description, URDF)
Before this commit: robot bimanual_shadowhand_motor, 32 links, 31 joints
Joints:
- joint FFJ4: origin xyz=0.033 0 0.095 rpy=0 0 0 -> xyz=-0.033 0 0.095 rpy=0 0 0
- joint LFJ5: origin xyz=-0.033 0 0.02071 rpy=0 -0.9599 0 -> xyz=0.033 0 0.02071 rpy=0 -0.9599 0
- joint MFJ4: origin xyz=0.011 0 0.099 rpy=0 0 0 -> xyz=-0.011 0 0.099 rpy=0 0 0
- joint RFJ4: origin xyz=-0.011 0 0.095 rpy=0 0 0 -> xyz=0.011 0 0.095 rpy=0 0 0
- joint THJ5: origin xyz=0.034 -0.00858 0.029 rpy=-0.785398163397 0 -1.57079632679 -> xyz=-0.034 -0.00858 0.029 rpy=-0.785398163397 0 1.57079632679
- joint palm_to_imu: origin xyz=0.01785 0.00765 0.049125 rpy=-1.5707963 3.141592 0.0 -> xyz=-0.01785 0.00765 0.049125 rpy=-1.5707963 3.141592 0.0

Commit message: left hand usable version

File: assets/urdf/shadow_hand/shadow_hand_left.urdf (robot description, URDF)
Before this commit: robot bimanual_shadowhand_motor, 32 links, 31 joints
Joints:
- joint THJ3: axis 0 1 0 -> 0 -1 0
- joint THJ4: axis 0 1 0 -> 0 -1 0
- joint THJ5: axis 0 0 -1 -> 0 0 1
- joint world_joint: origin xyz=0.0 0.0 0.0 rpy=0.0 0.0 0.0 -> xyz=0.0 0.0 0.0 rpy=0.0 0.0 1.57079

File: assets/urdf/shadow_hand/shadow_hand_right.urdf (robot description, URDF)
Before this commit: robot bimanual_shadowhand_motor, 32 links, 31 joints
Joints:
- joint world_joint: origin xyz=0.0 0.0 0.0 rpy=0.0 0.0 0.0 -> xyz=0.0 0.0 0.0 rpy=0.0 0.0 1.57079

File: assets/urdf/shadow_hand/shadow_hand_right_corrected.urdf (robot description, URDF)
Before this commit: robot bimanual_shadowhand_motor, 32 links, 31 joints
Links:
- link ffdistal: geometry collision mesh filename=meshes/visual/f_distal/pst/f_distal_pst.dae scale=0.001 0.001 0.001; visual mesh filename=meshes/visual/f_distal/pst/f_distal_pst.dae scale=0.001 0.001 0.001
- link ffknuckle: geometry collision cylinder length=0.014 radius=0.007; visual mesh filename=meshes/visual/f_knuckle/f_knuckle_E3M5.dae scale=0.001 0.001 0.001
- link ffmiddle: geometry collision cylinder length=0.025 radius=0.007; collision sphere radius=0.007
- link ffproximal: geometry collision cylinder length=0.040 radius=0.007; visual mesh filename=meshes/visual/f_proximal/f_proximal_E3M5.dae scale=0.001 0.001 0.001
- link lfdistal: geometry collision mesh filename=meshes/visual/f_distal/pst/f_distal_pst.dae scale=0.001 0.001 0.001; visual mesh filename=meshes/visual/f_distal/pst/f_distal_pst.dae scale=0.001 0.001 0.001
- link lfknuckle: geometry collision cylinder length=0.014 radius=0.007; visual mesh filename=meshes/visual/f_knuckle/f_knuckle_E3M5.dae scale=0.001 0.001 0.001
- link lfmetacarpal: geometry visual mesh filename=meshes/visual/lf_metacarpal/lf_metacarpal_E3M5.dae scale=0.001 0.001 0.001
- link lfmiddle: geometry collision cylinder length=0.025 radius=0.007; collision sphere radius=0.007
- link lfproximal: geometry collision cylinder length=0.040 radius=0.007; visual mesh filename=meshes/visual/f_proximal/f_proximal_E3M5.dae scale=0.001 0.001 0.001
- link mfdistal: geometry collision mesh filename=meshes/visual/f_distal/pst/f_distal_pst.dae scale=0.001 0.001 0.001; visual mesh filename=meshes/visual/f_distal/pst/f_distal_pst.dae scale=0.001 0.001 0.001
- link mfknuckle: geometry collision cylinder length=0.014 radius=0.007; visual mesh filename=meshes/visual/f_knuckle/f_knuckle_E3M5.dae scale=0.001 0.001 0.001
- link mfmiddle: geometry collision cylinder length=0.025 radius=0.007; collision sphere radius=0.007
- link mfproximal: geometry collision cylinder length=0.040 radius=0.007; visual mesh filename=meshes/visual/f_proximal/f_proximal_E3M5.dae scale=0.001 0.001 0.001
- link palm: geometry collision box size=0.018 0.024 0.004; collision box size=0.020 0.024 0.040
- link rfdistal: geometry collision mesh filename=meshes/visual/f_distal/pst/f_distal_pst.dae scale=0.001 0.001 0.001; visual mesh filename=meshes/visual/f_distal/pst/f_distal_pst.dae scale=0.001 0.001 0.001
- link rfknuckle: geometry collision cylinder length=0.014 radius=0.007; visual mesh filename=meshes/visual/f_knuckle/f_knuckle_E3M5.dae scale=0.001 0.001 0.001
- link rfmiddle: geometry collision cylinder length=0.025 radius=0.007; collision sphere radius=0.007
- link rfproximal: geometry collision cylinder length=0.040 radius=0.007; visual mesh filename=meshes/visual/f_proximal/f_proximal_E3M5.dae scale=0.001 0.001 0.001
- link thbase: geometry collision sphere radius=0.011; visual box size=0.001 0.001 0.001
- link thdistal: geometry collision mesh filename=meshes/visual/th_distal/pst/th_distal_pst.dae scale=0.001 0.001 0.001; visual mesh filename=meshes/visual/th_distal/pst/th_distal_pst.dae scale=0.001 0.001 0.001
- link thhub: geometry collision sphere radius=0.010; visual box size=0.001 0.001 0.001
- link thmiddle: geometry collision cylinder length=0.014 radius=0.010; collision cylinder length=0.018 radius=0.011
- link thproximal: geometry collision cylinder length=0.018 radius=0.012; visual mesh filename=meshes/visual/th_proximal/th_proximal_E3M5.dae scale=0.001 0.001 0.001
Joints:
- joint FFJ4: axis 0 -1 0 -> 0 1 0
- joint MFJ4: axis 0 -1 0 -> 0 1 0
- joint THJ1: axis 1 0 0 -> -1 0 0; limit lower=0.0 upper=1.57079632679 effort=1.0 velocity=4.0 -> lower=-1.57079632679 upper=0.0 effort=1.0 velocity=4.0
- joint THJ2: axis 1 0 0 -> -1 0 0

Commit message: mirroed left and right

File: assets/urdf/shadow_hand/shadow_hand_left.urdf (robot description, URDF)
Before this commit: robot bimanual_shadowhand_motor, 32 links, 31 joints
Links:
- link lfmetacarpal: geometry visual mesh filename=meshes/visual/lf_metacarpal/lf_metacarpal_E3M5_left.dae scale=0.001 0.001 0.001
Joints:
- joint LFJ4: axis 0 1 0 -> 0 -1 0; origin xyz=0.05397275 0 0.03779463 rpy=0 0.9599 0 -> xyz=0 0 0.06579 rpy=0 0 0
- joint LFJ5: axis 0 0 -1 -> 0.573576436 0 -0.819152044; origin xyz=0.033 0 0.02071 rpy=0 -0.9599 0 -> xyz=0.033 0 0.02071 rpy=0 0 0
- joint RFJ4: axis 0 1 0 -> 0 -1 0
- joint THJ1: axis 1 0 0 -> -1 0 0; limit lower=0.0 upper=1.57079632679 effort=1.0 velocity=4.0 -> lower=-1.57079632679 upper=0.0 effort=1.0 velocity=4.0
- joint THJ2: axis 1 0 0 -> -1 0 0; limit lower=-0.524 upper=0.524 effort=2.0 velocity=2.0 -> lower=-1.524 upper=1.524 effort=2.0 velocity=2.0

File: assets/urdf/shadow_hand/shadow_hand_right.urdf (robot description, URDF)
Before this commit: robot bimanual_shadowhand_motor, 32 links, 31 joints
Links:
- link lfmetacarpal: geometry visual mesh filename=meshes/visual/lf_metacarpal/lf_metacarpal_E3M5.dae scale=0.001 0.001 0.001
Joints:
- joint FFJ4: axis 0 -1 0 -> 0 1 0
- joint LFJ4: origin xyz=0.05397275 0 0.03779463 rpy=0 0.9599 0 -> xyz=0 0 0.06579 rpy=0 0 0
- joint LFJ5: axis 0 1 0 -> 0.573576436 0 0.819152044; origin xyz=-0.033 0 0.02071 rpy=0 -0.9599 0 -> xyz=-0.033 0 0.02071 rpy=0 0 0
- joint MFJ4: axis 0 -1 0 -> 0 1 0
- joint THJ1: axis 1 0 0 -> -1 0 0; limit lower=0.0 upper=1.57079632679 effort=1.0 velocity=4.0 -> lower=-1.57079632679 upper=0.0 effort=1.0 velocity=4.0
- joint THJ2: axis 1 0 0 -> -1 0 0
