Commit message: update

File: assets/mjcf/bucket/100454/mobility.urdf (robot description, URDF)
Before this commit: robot partnet_75612c0c1d5730eaf93a86670701266, 2 links, 1 joints
Joints:
- joint joint_1: origin xyz=0 0 0 rpy=1.570796326794897 0 -1.570796326794897 -> xyz=0 0 0.0 rpy=1.570796326794897 0 -1.570796326794897
